Commit message: modified:   urdf/r2d2.urdf

File: urdf/r2d2.urdf (robot description, URDF)
Before this commit: robot visual, 1 links, 0 joints
Links:
- link base_link: geometry visual mesh filename=package://testbot/meshes/Base.dae

Commit message: modified:   urdf/r2d2.urdf

File: urdf/r2d2.urdf (robot description, URDF)
Before this commit: robot visual, 1 links, 0 joints
Links:
- added link wheel_r; visual mesh filename=package://testbot/meshes/Rad_gelb.dae
Joints:
- added joint base_to_wheel_r: type fixed, parent base_link, child wheel_r, origin xyz=0 -0.25 0

Commit message: modified:   r2d2.urdf

File: urdf/r2d2.urdf (robot description, URDF)
Before this commit: robot visual, 2 links, 1 joints
Links:
- added link einhausung; visual mesh filename=package://testbot/meshes/Einhausung.dae
- added link wheel_l; visual mesh filename=package://testbot/meshes/Rad_gelb.dae
Joints:
- added joint base_to_einhausung: type fixed, parent base_link, child einhausung, origin xyz=-0.145 0 0.005
- added joint base_to_wheel_l: type fixed, parent base_link, child wheel_l, origin xyz=0 0.19 0.05
- joint base_to_wheel_r: origin xyz=0 -0.25 0 -> xyz=0 -0.19 0.05

Commit message: add stützrad mesh

File: urdf/r2d2.urdf (robot description, URDF)
Before this commit: robot visual, 4 links, 3 joints
Links:
- added link stuetz; visual mesh filename=package://testbot/meshes/Stuetzrad.dae
Joints:
- added joint base_to_stuetz: type fixed, parent base_link, child stuetz, origin xyz=-0.145 0 0.046

Commit message: Update r2d2.urdf

File: urdf/r2d2.urdf (robot description, URDF)
Before this commit: robot visual, 5 links, 4 joints
Joints:
- joint base_to_stuetz: origin xyz=-0.145 0 0.046 -> xyz=-0.145 0 0.051

Commit message: Update r2d2.urdf

File: urdf/r2d2.urdf (robot description, URDF)
Before this commit: robot visual, 5 links, 4 joints
Joints:
- joint base_to_stuetz: origin xyz=-0.145 0 0.051 -> xyz=-0.145 0 0.049

Commit message: add dome mesh

File: urdf/r2d2.urdf (robot description, URDF)
Before this commit: robot visual, 5 links, 4 joints
Links:
- added link dome; visual mesh filename=package://testbot/meshes/dome.dae
Joints:
- added joint base_to_dome: type fixed, parent base_link, child dome, origin xyz=0 0 0.005

Commit message: Update r2d2.urdf

File: urdf/r2d2.urdf (robot description, URDF)
Before this commit: robot visual, 6 links, 5 joints
Links:
- added link kinect; visual mesh filename=package://testbot/meshes/Kinect.dae
Joints:
- added joint dome_to_kinect: type fixed, parent dome, child kinect, origin xyz=0 0 0.25

Commit message: Update r2d2.urdf

File: urdf/r2d2.urdf (robot description, URDF)
Before this commit: robot visual, 7 links, 6 joints
Links:
- link stuetz: geometry visual mesh filename=package://testbot/meshes/lenkrolle.dae

Commit message: Update r2d2.urdf

File: urdf/r2d2.urdf (robot description, URDF)
Before this commit: robot visual, 7 links, 6 joints
Links:
- link stuetz: geometry visual mesh filename=package://testbot/meshes/Stuetzrad.dae

Commit message: modified:   r2d2.urdf

File: urdf/r2d2.urdf (robot description, URDF)
Before this commit: robot visual, 7 links, 6 joints
Links:
- link base_link: mass None -> 1.0; geometry collision mesh filename=package://testbot/meshes/Base.dae; visual mesh filename=package://testbot/meshes/Base.dae
- link dome: mass None -> 1.0; geometry collision mesh filename=package://testbot/meshes/dome.dae; visual mesh filename=package://testbot/meshes/dome.dae
- link einhausung: mass None -> 1.0; geometry collision mesh filename=package://testbot/meshes/Einhausung.dae; visual mesh filename=package://testbot/meshes/Einhausung.dae
- link kinect: mass None -> 1.0; geometry collision mesh filename=package://testbot/meshes/Kinect.dae; visual mesh filename=package://testbot/meshes/Kinect.dae
- link stuetz: mass None -> 1.0; geometry collision mesh filename=package://testbot/meshes/Stuetzrad.dae; visual mesh filename=package://testbot/meshes/Stuetzrad.dae
- link wheel_l: mass None -> 1.0; geometry collision mesh filename=package://testbot/meshes/Rad_gelb.dae; visual mesh filename=package://testbot/meshes/Rad_gelb.dae
- link wheel_r: mass None -> 1.0; geometry collision mesh filename=package://testbot/meshes/Rad_gelb.dae; visual mesh filename=package://testbot/meshes/Rad_gelb.dae

Commit message: modified:   r2d2.urdf

File: urdf/r2d2.urdf (robot description, URDF)
Before this commit: robot visual, 7 links, 6 joints
Links:
- link base_link: mass 1.0 -> 1.5
- link dome: mass 1.0 -> 0.5
- link kinect: mass 1.0 -> 0.3
- link stuetz: mass 1.0 -> 0.2
- link wheel_l: mass 1.0 -> 0.2
- link wheel_r: mass 1.0 -> 0.2
Joints:
- joint base_to_wheel_l: origin xyz=0 0.19 0.05 -> xyz=0 0.19 0.035
- joint base_to_wheel_r: origin xyz=0 -0.19 0.05 -> xyz=0 -0.19 0.035

Commit message: modified:   r2d2.urdf

File: urdf/r2d2.urdf (robot description, URDF)
Before this commit: robot visual, 7 links, 6 joints
Joints:
- joint base_to_wheel_l: axis (none) -> 0 1 0; type fixed -> continuous
- joint base_to_wheel_r: axis (none) -> 0 1 0; type fixed -> continuous
